File: Taller Arrancador EAGLE V1.0.0.brd (EAGLE design)
At the start: 18.4 x 13.3 mm, 15 parts, among them IC1 VS1838BB, U1 ATTINY25/45/85

Commit message: Add files via upload
Parts:
- removed JP2: (no value), pinhead-2:1X02-S
- removed R4, R5: 330E, rcl:R0603
- removed U1: ATTINY25/45/85, ATMEL-ATTINY25-45-85:TSSOP-8
- added C5: 0.1uF, rcl:C0603
- added GOLD_ORB_SM1: OSHWLOGOLOGO5MM, oshw:OSHW_5MM
- added U2: ATTINY412-SSNR, Attiny412-serie-tiny-0:SOIC8_SA_SST_MCH
- R3: value 10K -> 1.2k
- moved C1 11.3 mm to (4.80, 9.00), turned to 90 degrees
- moved LED1 3.68 mm to (13.8, 11.3), turned to 270 degrees
- moved R3 3.25 mm to (14.0, 7.80)
- moved C3 2.48 mm to (14.1, 6.14), turned to 180 degrees
- moved C2 1.94 mm to (13.9, 3.02), turned to 180 degrees
- moved R1 1.88 mm to (7.19, 4.28)
- moved LED2 1.01 mm to (13.8, 9.91), turned to 270 degrees
- moved R2 0.81 mm to (4.38, 4.21)
- moved C4 0.05 mm to (8.91, 3.12), turned to 0 degrees
Connections:
- removed net N$4: LED1.C, R4.2
- removed net N$5: JP2.1, R3.1, U1.1
- removed net N$8: JP1.4, U1.5
- removed net N$9: JP1.3, U1.6
- new net SEÑAL: JP1.3, U2.3
- new net UPDI: JP1.4, U2.6
- net +5V: now also C5.1, JP1.2, U2.1; no longer JP1.1, R3.2, U1.8
- net GND: now also C5.2, JP1.1, R3.2, U2.8; no longer JP1.2, R4.1, R5.1, U1.4
- net N$3: now also U2.5; no longer U1.2
- net N$6: now also U2.7; no longer U1.3
- net N$7: now also LED1.C, R3.1; no longer R5.2
- net OUT: now also U2.4; no longer JP2.2, U1.7
Routing:
- net N$8: track 21.4 -> 0.00 mm, vias 1 -> 0
- net +5V: track 28.8 -> 10.9 mm, vias 2 -> 0
- net UPDI: track 0.00 -> 13.2 mm, vias 0 -> 1
- net N$9: track 12.3 -> 0.00 mm, vias 1 -> 0
- net SEÑAL: track 0.00 -> 10.4 mm, vias 0 -> 1
- net GND: track 40.0 -> 31.4 mm, vias 2 -> 1
- net N$5: track 8.06 -> 0.00 mm, vias 1 -> 0
- net N$1: track 11.4 -> 16.5 mm, vias 0 -> 1
- net N$6: track 2.80 -> 7.75 mm
- net N$4: track 1.73 -> 0.00 mm
- net N$7: track 2.45 -> 3.60 mm
- net N$3: track 4.12 -> 3.18 mm
- net OUT: track 12.0 -> 12.5 mm, vias 0 -> 1
Other:
- board size 18.4 x 13.3 mm -> 17.3 x 13.3 mm
- board text added: "Diseñado en México por Sol y Nomada-e"

Commit message: Add files via upload
Parts:
- removed C4: 10uF, rcl:C0603
- removed IC1: VS1838BB, LFN-VS1838B_Infrared_Sensor:VS1838B
- removed R1: 100E, rcl:R0603
- added U1: TSOP75338WTT, receptorir38:TSOP75338WTT_VIS
- C2: value 100uF -> 0.1uF; device rcl:CT3216 -> rcl:C0402
- C3: device rcl:C0603 -> rcl:C0402
- R2: value 22K -> 100
- moved C2 2.52 mm to (13.5, 5.50), turned to 90 degrees
- moved C3 2.17 mm to (12.0, 5.50), turned to 90 degrees
- moved GOLD_ORB_SM1 1.77 mm to (12.3, 4.90)
- moved R2 1.22 mm to (4.10, 5.40)
Connections:
- removed net N$1: C2.+, C3.1, C4.1, IC1.VCC, R1.1
- new net N$2: C2.1, C3.1, R2.1, U1.2
- net +5V: no longer R1.2
- net GND: now also C2.2, U1.1, U1.4; no longer C2.-, C4.2, IC1.GND
- net OUT: now also U1.3; no longer IC1.OUT, R2.1
Routing:
- net N$1: track 16.5 -> 0.00 mm, vias 1 -> 0
- net N$2: track 0.00 -> 15.8 mm
- net OUT: track 12.5 -> 4.72 mm, vias 1 -> 0
- net GND: track 31.4 -> 36.1 mm, vias 1 -> 2
- net +5V: track 10.9 -> 9.78 mm
Other:
- board size 17.3 x 13.3 mm -> 16 x 13.3 mm
- board text added: "C:/Users/SYSTEMS/Downloads/logo.bmp"
- board text added: "Diseñado en Méixco por Sol"
- board text added: "y Nomada-e"
- board text removed: "Diseñado en México por Sol y Nomada-e"
