File: Taller Arrancador EAGLE V1.0.0.sch (EAGLE design)
At the start: 15 parts, among them IC1 VS1838BB, U1 ATTINY25/45/85

Commit message: Add files via upload
Parts:
- removed JP2: (no value), pinhead-2:PINHD-1X02_2.54-S
- removed R4, R5: 330E, rcl:R-US_R0603
- removed U1: ATTINY25/45/85, ATMEL-ATTINY25-45-85:ATTINY25/45/85
- added C5: 0.1uF, rcl:C-EUC0603
- added GOLD_ORB_SM1: OSHWLOGOLOGO5MM, oshw:OSHWLOGOLOGO5MM
- added U2: ATTINY412-SSNR, Attiny412-serie-tiny-0:ATTINY412-SSNR
- R3: value 10K -> 1.2k; device rcl:R-US_R0603 -> rcl:R-EU_R0603
Connections:
- removed net N$4: LED1.C, R4.2
- removed net N$5: JP2.1, R3.1, U1.PB5(RESET)
- removed net N$8: JP1.4, U1.PB0(MOSI/OC0A/OC1A)
- removed net N$9: JP1.3, U1.PB1(MISO/OC0B/OC0A)
- new net SEÑAL: JP1.3, U2.PA7
- new net UPDI: JP1.4, U2.PA0/!RESET/UPDI
- net +5V: now also C5.1, JP1.2, U2.VDD; no longer JP1.1, R3.2, U1.VCC
- net GND: now also C5.2, JP1.1, R3.2, U2.GND; no longer JP1.2, R4.1, R5.1, U1.GND
- net N$3: now also U2.PA2; no longer U1.PB3(XTAL1/OC1B)
- net N$6: now also U2.PA3/EXTCLK; no longer U1.PB4(XTAL2/OC1B)
- net N$7: now also LED1.C, R3.1; no longer R5.2
- net OUT: now also U2.PA1; no longer JP2.2, U1.PB2(SCK)

Commit message: Add files via upload
Parts:
- removed C4: 10uF, rcl:C-EUC0603
- removed IC1: VS1838BB, LFN-VS1838B_Infrared_Sensor:VS1838BB
- removed R1: 100E, rcl:R-US_R0603
- added U1: TSOP75338WTT, receptorir38:TSOP75338WTT
- C2: value 100uF -> 0.1uF; device rcl:CPOL-EUCT3216 -> rcl:C-EUC0402
- C3: device rcl:C-EUC0603 -> rcl:C-EUC0402
- R2: value 22K -> 100; device rcl:R-US_R0603 -> rcl:R-EU_R0603
Connections:
- removed net N$1: C2.+, C3.1, C4.1, IC1.VCC, R1.1
- new net N$2: C2.1, C3.1, R2.1, U1.VS
- net +5V: no longer R1.2
- net GND: now also C2.2, U1.GND, U1.GND_2; no longer C2.-, C4.2, IC1.GND
- net OUT: now also U1.OUT; no longer IC1.OUT, R2.1
Other:
- moved on the sheet: C3
